Commit message: added inertia tag to the box body

File: urdf/common_properties.xacro (robot description, xacro)
@@ -7,3 +7,10 @@
         <color rgba="0.5 0.5 0.5 1"/>
     </material>
+    <xacro:macro name="box_inertia" params="m l w h xyz rpy">
+        <inertial>
+            <origin xyz="${xyz}" rpy="${rpy}"/>
+            <mass value="${m}"/>
+            <inertia ixx="${(m/12)*((h*h)+(l*l)}" ixy="0.0" ixz="0.0" iyy="${(m/12)*((w*w)+(l*l)}" iyz="0.0" izz="${(m/12)*((w*w)+(h*h)}"/>
+        </inertial>
+    </xacro:macro>
 </robot>

File: urdf/mobile_base.xacro (robot description, xacro)
@@ -19,4 +19,5 @@
             <material name="green"/>
         </visual>
+        <xacro:box_inertia m="5.0" l="${base_length}" w="${base_width}" h="${base_height}" xyz="0 0 ${base_height / 2}" rpy="0 0 0" />
     </link>
     <xacro:macro name="wheel_link" params="prefix">

Commit message: inertia+gazebo integration update

File: urdf/common_properties.xacro (robot description, xacro)
@@ -11,5 +11,19 @@
             <origin xyz="${xyz}" rpy="${rpy}"/>
             <mass value="${m}"/>
-            <inertia ixx="${(m/12)*((h*h)+(l*l)}" ixy="0.0" ixz="0.0" iyy="${(m/12)*((w*w)+(l*l)}" iyz="0.0" izz="${(m/12)*((w*w)+(h*h)}"/>
+            <inertia ixx="${(m/12)*((h*h)+(l*l))}" ixy="0.0" ixz="0.0" iyy="${(m/12)*((w*w)+(l*l))}" iyz="0.0" izz="${(m/12)*((w*w)+(h*h))}"/>
+        </inertial>
+    </xacro:macro>
+    <xacro:macro name="wheel_inertia" params="m r h xyz rpy">
+        <inertial>
+            <origin xyz="${xyz}" rpy="${rpy}"/>
+            <mass value="${m}"/>
+            <inertia ixx="${(m/12)*((3*r*r)+(h*h))}" ixy="0.0" ixz="0.0" iyy="${(m/12)*((3*r*r)+(h*h))}" iyz="0.0" izz="${((m*r*r)/2)}"/>
+        </inertial>
+    </xacro:macro>
+    <xacro:macro name="ball_inertia" params="m r xyz rpy">
+        <inertial>
+            <origin xyz="${xyz}" rpy="${rpy}"/>
+            <mass value="${m}"/>
+            <inertia ixx="${(2/5)*m*(r*r)}" ixy="0.0" ixz="0.0" iyy="${(2/5)*m*(r*r)}" iyz="0.0" izz="${(2/5)*m*(r*r)}"/>
         </inertial>
     </xacro:macro>

File: urdf/mobile_base.xacro (robot description, xacro)
@@ -19,5 +19,11 @@
             <material name="green"/>
         </visual>
-        <xacro:box_inertia m="5.0" l="${base_length}" w="${base_width}" h="${base_height}" xyz="0 0 ${base_height / 2}" rpy="0 0 0" />
+        <collision>
+            <geometry>
+                <box size="${base_length} ${base_width} ${base_height}"></box>
+            </geometry>
+            <origin xyz="0 0 ${base_height / 2}" rpy="0 0 0"></origin>
+        </collision>
+        <xacro:box_inertia m="5.0" l="${2*base_length}" w="${2*base_width}" h="${2*base_height}" xyz="0 0 ${base_height / 2}" rpy="0 0 0" />
     </link>
     <xacro:macro name="wheel_link" params="prefix">
@@ -30,4 +36,11 @@
                 <material name="gray"/>
             </visual>
+            <collision>
+                <geometry>
+                    <cylinder radius="${wheel_radius}" length="${wheel_length}"/>
+                </geometry>
+                <origin xyz="0 0 0" rpy="0 0 0"></origin>
+            </collision>
+            <xacro:wheel_inertia m="1.0" r="${2*wheel_radius}" h="${2*wheel_length}" xyz="0 0 0" rpy="0 0 0" />
         </link>
     </xacro:macro>
@@ -42,4 +55,11 @@
             <material name="gray"/>
         </visual>
+        <collision>
+            <geometry>
+                <sphere radius="${wheel_radius / 2}"/>
+            </geometry>
+            <origin xyz="0 0 0" rpy="0 0 0"></origin>
+        </collision>
+        <xacro:ball_inertia m="0.5" r="${2*wheel_radius / 2}" xyz="0 0 0" rpy="0 0 0" />
     </link>
     <joint name="base_right_wheel_joint" type="continuous">

File: urdf/my_robot.urdf.xacro (robot description, xacro)
@@ -3,3 +3,4 @@
     <xacro:include filename="common_properties.xacro"/>
     <xacro:include filename="mobile_base.xacro"/>
+    <xacro:include filename="mobile_base_gazebo.xacro"/>
 </robot>

Commit message: final project update

File: urdf/common_properties.xacro (robot description, xacro)
@@ -2,28 +2,40 @@
 <robot xmlns:xacro="http://www.ros.org/wiki/xacro">
     <material name="green">
-        <color rgba="0.0 0.5 0.0 1"/>
+        <color rgba="0 0.5 0 1" />
     </material>
-    <material name="gray">
-        <color rgba="0.5 0.5 0.5 1"/>
+    <material name="grey">
+        <color rgba="0.5 0.5 0.5 1" />
+    </material>
+    <material name="orange">
+        <color rgba="1.0 0.5 0 1" />
+    </material>
+    <material name="yellow">
+        <color rgba="1.0 1.0 0 1" />
     </material>
     <xacro:macro name="box_inertia" params="m l w h xyz rpy">
         <inertial>
-            <origin xyz="${xyz}" rpy="${rpy}"/>
-            <mass value="${m}"/>
-            <inertia ixx="${(m/12)*((h*h)+(l*l))}" ixy="0.0" ixz="0.0" iyy="${(m/12)*((w*w)+(l*l))}" iyz="0.0" izz="${(m/12)*((w*w)+(h*h))}"/>
+            <origin xyz="${xyz}" rpy="${rpy}" />
+            <mass value="${m}" />
+            <inertia ixx="${(m/12) * (h*h + l*l)}" ixy="0" ixz="0"
+                     iyy="${(m/12) * (w*w + l*l)}" iyz="0"
+                     izz="${(m/12) * (w*w + h*h)}" />
         </inertial>
     </xacro:macro>
-    <xacro:macro name="wheel_inertia" params="m r h xyz rpy">
+    <xacro:macro name="cylinder_inertia" params="m r h xyz rpy">
         <inertial>
-            <origin xyz="${xyz}" rpy="${rpy}"/>
-            <mass value="${m}"/>
-            <inertia ixx="${(m/12)*((3*r*r)+(h*h))}" ixy="0.0" ixz="0.0" iyy="${(m/12)*((3*r*r)+(h*h))}" iyz="0.0" izz="${((m*r*r)/2)}"/>
+            <origin xyz="${xyz}" rpy="${rpy}" />
+            <mass value="${m}" />
+            <inertia ixx="${(m/12) * (3*r*r + h*h)}" ixy="0" ixz="0"
+                     iyy="${(m/12) * (3*r*r + h*h)}" iyz="0"
+                     izz="${(m/2) * (r*r)}" />
         </inertial>
     </xacro:macro>
-    <xacro:macro name="ball_inertia" params="m r xyz rpy">
+    <xacro:macro name="sphere_inertia" params="m r xyz rpy">
         <inertial>
-            <origin xyz="${xyz}" rpy="${rpy}"/>
-            <mass value="${m}"/>
-            <inertia ixx="${(2/5)*m*(r*r)}" ixy="0.0" ixz="0.0" iyy="${(2/5)*m*(r*r)}" iyz="0.0" izz="${(2/5)*m*(r*r)}"/>
+            <origin xyz="${xyz}" rpy="${rpy}" />
+            <mass value="${m}" />
+            <inertia ixx="${(2/5) * m * r * r}" ixy="0" ixz="0"
+                     iyy="${(2/5) * m * r * r}" iyz="0"
+                     izz="${(2/5) * m * r * r}" />
         </inertial>
     </xacro:macro>

File: urdf/mobile_base.xacro (robot description, xacro)
@@ -1,29 +1,26 @@
 <?xml version="1.0"?>
 <robot xmlns:xacro="http://www.ros.org/wiki/xacro">
-    <xacro:property name="base_length" value="0.6"/>
-    <xacro:property name="base_width" value="0.4"/>
-    <xacro:property name="base_height" value="0.2"/>
-    <xacro:property name="wheel_radius" value="0.1"/>
-    <xacro:property name="wheel_length" value="0.05"/>
-    <link name="footprint_link">
-        <visual>
-            <origin xyz="0 0 0" rpy="0 0 0"></origin>
-        </visual>
-    </link>
+    <xacro:property name="base_length" value="0.6" />
+    <xacro:property name="base_width" value="0.4" />
+    <xacro:property name="base_height" value="0.2" />
+    <xacro:property name="wheel_radius" value="0.1" />
+    <xacro:property name="wheel_length" value="0.05" />
+    <link name="base_footprint" />
     <link name="base_link">
         <visual>
             <geometry>
-                <box size="${base_length} ${base_width} ${base_height}"></box>
+                <box size="${base_length} ${base_width} ${base_height}" />
             </geometry>
-            <origin xyz="0 0 ${base_height / 2}" rpy="0 0 0"></origin>
-            <material name="green"/>
+            <origin xyz="0 0 ${base_height / 2.0}" rpy="0 0 0" />
+            <material name="green" />
         </visual>
         <collision>
             <geometry>
-                <box size="${base_length} ${base_width} ${base_height}"></box>
+                <box size="${base_length} ${base_width} ${base_height}" />
             </geometry>
-            <origin xyz="0 0 ${base_height / 2}" rpy="0 0 0"></origin>
+            <origin xyz="0 0 ${base_height / 2.0}" rpy="0 0 0" />
         </collision>
-        <xacro:box_inertia m="5.0" l="${2*base_length}" w="${2*base_width}" h="${2*base_height}" xyz="0 0 ${base_height / 2}" rpy="0 0 0" />
+        <xacro:box_inertia m="5.0" l="${2*base_length}" w="${2*base_width}" h="${2*base_height}"
+                           xyz="0 0 ${base_height / 2.0}" rpy="0 0 0" />
     </link>
     <xacro:macro name="wheel_link" params="prefix">
@@ -31,57 +28,59 @@
             <visual>
                 <geometry>
-                    <cylinder radius="${wheel_radius}" length="${wheel_length}"/>
+                    <cylinder radius="${wheel_radius}" length="${wheel_length}" />
                 </geometry>
-                <origin xyz="0 0 0" rpy="0 0 0"></origin>
-                <material name="gray"/>
+                <origin xyz="0 0 0" rpy="${pi / 2.0} 0 0" />
+                <material name="grey" />
             </visual>
             <collision>
                 <geometry>
-                    <cylinder radius="${wheel_radius}" length="${wheel_length}"/>
+                    <cylinder radius="${wheel_radius}" length="${wheel_length}" />
                 </geometry>
-                <origin xyz="0 0 0" rpy="0 0 0"></origin>
+                <origin xyz="0 0 0" rpy="${pi / 2.0} 0 0" />
             </collision>
-            <xacro:wheel_inertia m="1.0" r="${2*wheel_radius}" h="${2*wheel_length}" xyz="0 0 0" rpy="0 0 0" />
+            <xacro:cylinder_inertia m="1.0" r="${2*wheel_radius}" h="${2*wheel_length}"
+                                    xyz="0 0 0" rpy="${pi / 2.0} 0 0" />
         </link>
     </xacro:macro>
-    <xacro:wheel_link prefix="right"/>
-    <xacro:wheel_link prefix="left"/>
-    <link name="caster_wheel">
+    <xacro:wheel_link prefix="right" />
+    <xacro:wheel_link prefix="left" />
+    <link name="caster_wheel_link">
         <visual>
             <geometry>
-                <sphere radius="${wheel_radius / 2}"/>
+                <sphere radius="${wheel_radius / 2.0}" />
             </geometry>
-            <origin xyz="0 0 0" rpy="0 0 0"></origin>
-            <material name="gray"/>
+            <origin xyz="0 0 0" rpy="0 0 0" />
+            <material name="grey" />
         </visual>
         <collision>
             <geometry>
-                <sphere radius="${wheel_radius / 2}"/>
+                <sphere radius="${wheel_radius / 2.0}" />
             </geometry>
-            <origin xyz="0 0 0" rpy="0 0 0"></origin>
+            <origin xyz="0 0 0" rpy="0 0 0" />
         </collision>
-        <xacro:ball_inertia m="0.5" r="${2*wheel_radius / 2}" xyz="0 0 0" rpy="0 0 0" />
+        <xacro:sphere_inertia m="0.5" r="${2*wheel_radius / 2.0}"
+                              xyz="0 0 0" rpy="0 0 0" />
     </link>
+    <joint name="base_joint" type="fixed">
+        <parent link="base_footprint" />
+        <child link="base_link" />
+        <origin xyz="0 0 ${wheel_radius}" rpy="0 0 0"/>
+    </joint>
     <joint name="base_right_wheel_joint" type="continuous">
-        <parent link="base_link"/>
-        <child link="right_wheel_link"/>
-        <origin xyz="${-base_length / 4.0} ${-(base_width+wheel_length)/2} 0.0" rpy="${pi / 2.0} 0.0 0.0"/>
-        <axis xyz="0.0 0.0 -1"/>
+        <parent link="base_link" />
+        <child link="right_wheel_link" />
+        <origin xyz="${-base_length / 4.0} ${-(base_width + wheel_length) / 2.0} 0" rpy="0 0 0" />
+        <axis xyz="0 1 0" />
     </joint>
     <joint name="base_left_wheel_joint" type="continuous">
-        <parent link="base_link"/>
-        <child link="left_wheel_link"/>
-        <origin xyz="${-base_length / 4.0} ${(base_width+wheel_length)/2} 0.0" rpy="${pi / 2.0} 0.0 0.0"/>
-        <axis xyz="0.0 0.0 -1"/>
+        <parent link="base_link" />
+        <child link="left_wheel_link" />
+        <origin xyz="${-base_length / 4.0} ${(base_width + wheel_length) / 2.0} 0" rpy="0 0 0" />
+        <axis xyz="0 1 0" />
     </joint>
     <joint name="base_caster_wheel_joint" type="fixed">
-        <origin xyz="${base_length/3.0} 0.0 ${-wheel_radius/2}" rpy="0.0 0.0 0.0"/>
-        <parent link="base_link"/>
-        <child link="caster_wheel"/>
-    </joint>
-    <joint name="base_footprint_joint" type="fixed">
-        <origin xyz="0.0 0.0 ${wheel_radius}" rpy="0.0 0.0 0.0"/>
-        <parent link="footprint_link"/>
-        <child link="base_link"/>
+        <parent link="base_link" />
+        <child link="caster_wheel_link" />
+        <origin xyz="${base_length / 3.0} 0 ${-wheel_radius / 2.0}" rpy="0 0 0" />
     </joint>
 </robot>

File: urdf/mobile_base_gazebo.xacro (robot description, xacro)
@@ -2,24 +2,16 @@
 <robot xmlns:xacro="http://www.ros.org/wiki/xacro">
     <gazebo reference="base_link">
-        <material>
-            Gazebo/Green
-        </material>
+        <material>Gazebo/Green</material>
     </gazebo>
     <gazebo reference="right_wheel_link">
-        <material>
-            Gazebo/Gray
-        </material>
+        <material>Gazebo/Grey</material>
     </gazebo>
     <gazebo reference="left_wheel_link">
-        <material>
-            Gazebo/Gray
-        </material>
+        <material>Gazebo/Grey</material>
     </gazebo>
-    <gazebo reference="caster_wheel">
-        <material>
-            Gazebo/Gray
-        </material>
-        <mu1 value="0.1"/>
-        <mu2 value="0.1"/>
+    <gazebo reference="caster_wheel_link">
+        <material>Gazebo/Grey</material>
+        <mu1 value="0.1" />
+        <mu2 value="0.1" />
     </gazebo>
     <gazebo>
@@ -39,6 +31,6 @@
             <odometry_topic>odom</odometry_topic>
             <odometry_frame>odom</odometry_frame>
-            <robot_base_frame>footprint_link</robot_base_frame>
-          </plugin>
+            <robot_base_frame>base_footprint</robot_base_frame>
+        </plugin>
     </gazebo>
 </robot>

File: urdf/my_robot.urdf.xacro (robot description, xacro)
@@ -1,6 +1,14 @@
 <?xml version="1.0"?>
 <robot name="my_robot" xmlns:xacro="http://www.ros.org/wiki/xacro">
-    <xacro:include filename="common_properties.xacro"/>
-    <xacro:include filename="mobile_base.xacro"/>
-    <xacro:include filename="mobile_base_gazebo.xacro"/>
+    <xacro:include filename="common_properties.xacro" />
+    <xacro:include filename="mobile_base.xacro" />
+    <xacro:include filename="mobile_base_gazebo.xacro" />
+    <xacro:include filename="arm.xacro" />
+    <xacro:include filename="arm_gazebo.xacro" />
+    <joint name="mobile_base_arm_joint" type="fixed">
+        <parent link="base_link" />
+        <child link="arm_base_link" />
+        <origin xyz="${base_length / 4.0} 0 ${base_height}" rpy="0 0 0" />
+    </joint>
+    <xacro:include filename="camera.xacro" />
 </robot>
